Commit message: Add turtlebot functionality and fix follow waypoints by stamped message

File: core_cleaning_robot/models/cleaning_robot/gazebo_control.xacro (robot description, xacro)
@@ -4,6 +4,6 @@
     <plugin name="ignition::gazebo::systems::DiffDrive" filename="libignition-gazebo-diff-drive-system.so">
         <!-- Wheel information-->
-        <left_joint>left_wheel_joint</left_joint>
-        <right_joint>right_wheel_joint</right_joint>
+        <left_joint>wheel_left_joint</left_joint>
+        <right_joint>wheel_right_joint</right_joint>
         <wheel_separation>0.35</wheel_separation>
         <wheel_radius>0.05</wheel_radius>
@@ -16,5 +16,5 @@
             <robot_base_frame>$(arg name)/base_link</robot_base_frame>
             <odom_publish_frequency>10</odom_publish_frequency>
-            <odom_topic>/model/$(arg name)/odometry_IMU</odom_topic>
+            <odom_topic>/model/$(arg name)/odometry</odom_topic>
             <odom_covariance_topic>/model/$(arg name)/odometry_with_covariance</odom_covariance_topic>
             <tf_topic>/model/$(arg name)/odometry_tf</tf_topic>

File: core_cleaning_robot/models/cleaning_robot/lidar.xacro (robot description, xacro)
@@ -15,8 +15,8 @@
     <joint name="lidar_joint" type="fixed">
         <parent link="chassis"/>
-        <child link="base_laser"/>
+        <child link="base_scan"/>
         <origin xyz="${$(arg length)/2} 0 0.01" rpy="0 0 0"/>
     </joint>
-    <link name="base_laser">
+    <link name="base_scan">
        <visual>
             <geometry>
@@ -34,5 +34,5 @@
         </xacro:inertial_cylinder>
     </link>
-    <gazebo reference= "base_laser">
+    <gazebo reference= "base_scan">
         <material>Gazebo/Red</material>
         <xacro:if value="$(arg laser_enable)">
@@ -43,5 +43,5 @@
             <pose>0 0 0 0 0 0</pose>
             <topic>/model/$(arg name)/scan</topic>
-            <ignition_frame_id>$(arg name)/base_laser</ignition_frame_id>
+            <ignition_frame_id>$(arg name)/base_scan</ignition_frame_id>
             <update_rate>10</update_rate>
             <ray>

File: core_cleaning_robot/models/cleaning_robot/robot_core.xacro (robot description, xacro)
@@ -58,5 +58,5 @@
     </gazebo>
     <!-- LEFT WHEEL LINK -->
-    <joint name="left_wheel_joint" type="continuous">
+    <joint name="wheel_left_joint" type="continuous">
         <parent link="base_link"/>
         <child link="left_wheel"/>
@@ -83,5 +83,5 @@
     </gazebo>
     <!-- RIGHT WHEEL LINK -->
-    <joint name="right_wheel_joint" type="continuous">
+    <joint name="wheel_right_joint" type="continuous">
         <parent link="base_link"/>
         <child link="right_wheel"/>

File: core_dynamical_agent/models/agent/lidar.xacro (robot description, xacro)
@@ -17,8 +17,8 @@
     <joint name="lidar_joint" type="fixed">
         <parent link="chassis"/>
-        <child link="base_laser"/>
+        <child link="base_scan"/>
         <origin xyz="0.1 0 0.125" rpy="0 0 0"/>
     </joint>
-    <link name="base_laser">
+    <link name="base_scan">
         <visual>
             <origin xyz="0 0 0" rpy="0 0 0"/>
@@ -37,5 +37,5 @@
         </xacro:inertial_cylinder>
     </link>
-    <gazebo reference= "base_laser">
+    <gazebo reference= "base_scan">
         <material>Gazebo/Red</material>
         <collision>
@@ -53,5 +53,5 @@
                 <pose>0 0 0 0 0 0</pose>
                 <topic>/model/$(arg name)/scan</topic>
-                <ignition_frame_id>$(arg name)/base_laser</ignition_frame_id>
+                <ignition_frame_id>$(arg name)/base_scan</ignition_frame_id>
                 <update_rate>10</update_rate>
                 <ray>
